File: angelia.kicad_pcb (KiCad board)
At the start: 2 copper layers, 160 x 120 mm, 261 parts, among them J10 Conn_Coaxial, J15 Conn_02x05_Top_Bottom, J16 Conn_02x13_Top_Bottom, J18 Conn_02x05_Top_Bottom, J25 Conn_Coaxial, J3 Conn_Coaxial, J5 Conn_Coaxial, J7 RJ45, P1 Conn_02x05_Top_Bottom, P2 Conn_02x05_Top_Bottom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

Commit message: ferrites and vlsi
Parts:
- removed U5: EP4CE115F780, Package_BGA:BGA-676_27.0x27.0mm_Layout26x26_P1.0mm_Ball0.6mm_Pad0.5mm_NSMD
- added J33: ATX-20, Connector_Molex:Molex_Mini-Fit_Jr_5566-20A_2x10_P4.20mm_Vertical, F.Cu at (116.6, 146.5)
- added L1: 220, Inductor_SMD:L_0805_2012Metric_Pad1.05x1.20mm_HandSolder, F.Cu at (234.2, 51.2)
- added L10: 220, Inductor_SMD:L_0805_2012Metric_Pad1.05x1.20mm_HandSolder, F.Cu at (239.1, 51.2)
- added L11: 220, Inductor_SMD:L_0805_2012Metric_Pad1.05x1.20mm_HandSolder, F.Cu at (239.1, 54.0)
- added L12: 220, Inductor_SMD:L_0805_2012Metric_Pad1.05x1.20mm_HandSolder, F.Cu at (239.1, 56.8)
- added L14: 220, Inductor_SMD:L_0805_2012Metric_Pad1.05x1.20mm_HandSolder, F.Cu at (239.1, 59.5)
- added L15: 220, Inductor_SMD:L_0805_2012Metric_Pad1.05x1.20mm_HandSolder, F.Cu at (239.1, 62.2)
- added L16: 220, Inductor_SMD:L_0805_2012Metric_Pad1.05x1.20mm_HandSolder, F.Cu at (239.1, 65.0)
- added L2: 220, Inductor_SMD:L_0805_2012Metric_Pad1.05x1.20mm_HandSolder, F.Cu at (234.2, 54.0)
- added L20: 220, Inductor_SMD:L_0805_2012Metric_Pad1.05x1.20mm_HandSolder, F.Cu at (239.1, 67.8)
- added L21: 220, Inductor_SMD:L_0805_2012Metric_Pad1.05x1.20mm_HandSolder, F.Cu at (244.0, 51.2)
- added L22: 220, Inductor_SMD:L_0805_2012Metric_Pad1.05x1.20mm_HandSolder, F.Cu at (244.0, 54.0)
- added L23: 220, Inductor_SMD:L_0805_2012Metric_Pad1.05x1.20mm_HandSolder, F.Cu at (244.0, 56.8)
- added L24: 220, Inductor_SMD:L_0805_2012Metric_Pad1.05x1.20mm_HandSolder, F.Cu at (244.0, 59.5)
- added L3: 560nH, Inductor_SMD:L_0805_2012Metric_Pad1.05x1.20mm_HandSolder, F.Cu at (163.4, 40.3)
- added L30: 220, Inductor_SMD:L_0805_2012Metric_Pad1.05x1.20mm_HandSolder, F.Cu at (244.0, 62.2)
- added L32: 220, Inductor_SMD:L_0805_2012Metric_Pad1.05x1.20mm_HandSolder, F.Cu at (244.0, 65.0)
- added L33: 220, Inductor_SMD:L_0805_2012Metric_Pad1.05x1.20mm_HandSolder, F.Cu at (244.0, 67.8)
- added L38: 220, Inductor_SMD:L_0805_2012Metric_Pad1.05x1.20mm_HandSolder, F.Cu at (248.8, 51.2)
- added L4: 22n, Inductor_SMD:L_0805_2012Metric_Pad1.05x1.20mm_HandSolder, F.Cu at (163.4, 44.9)
- added L41: 220, Inductor_SMD:L_0805_2012Metric_Pad1.05x1.20mm_HandSolder, F.Cu at (248.8, 54.0)
- added L42: 220, Inductor_SMD:L_0805_2012Metric_Pad1.05x1.20mm_HandSolder, F.Cu at (248.8, 56.8)
- added L43: 220, Inductor_SMD:L_0805_2012Metric_Pad1.05x1.20mm_HandSolder, F.Cu at (248.8, 59.5)
- added L44: 220, Inductor_SMD:L_0805_2012Metric_Pad1.05x1.20mm_HandSolder, F.Cu at (248.8, 62.2)
- added L45: 220, Inductor_SMD:L_0805_2012Metric_Pad1.05x1.20mm_HandSolder, F.Cu at (248.8, 65.0)
- added L6: 220, Inductor_SMD:L_0805_2012Metric_Pad1.05x1.20mm_HandSolder, F.Cu at (234.2, 62.2)
- added L8: 220, Inductor_SMD:L_0805_2012Metric_Pad1.05x1.20mm_HandSolder, F.Cu at (234.2, 65.0)
- added L9: 220, Inductor_SMD:L_0805_2012Metric_Pad1.05x1.20mm_HandSolder, F.Cu at (234.2, 67.8)
- added P3: EP4CE115F780, Package_BGA:BGA-676_27.0x27.0mm_Layout26x26_P1.0mm_Ball0.6mm_Pad0.5mm_NSMD, F.Cu at (136.9, 78.7)
- added U14: SN65LVDM180D, Package_SO:SOIC-14_3.9x8.7mm_P1.27mm, B.Cu at (175.2, 101.1)
- added U22: ULN2003A, Package_SO:SOIC-16W_5.3x10.2mm_P1.27mm, B.Cu at (200.4, 107.6)
- added U3: LMC6482AM, Package_SO:SO-8_5.3x6.2mm_P1.27mm, B.Cu at (128.8, 39.8)
- added U301: ~, Package_SO:TSOP-I-48_18.4x12mm_P0.5mm, F.Cu at (132.1, 105.8)
- added U4: LMC6482AM, Package_SO:SO-8_5.3x6.2mm_P1.27mm, B.Cu at (204.2, 45.9)
- added U6: OPA2674IC, Package_SO:SO-8_5.3x6.2mm_P1.27mm, F.Cu at (180.8, 43.8)
- added U7: OPA2674IC, Package_SO:SO-8_5.3x6.2mm_P1.27mm, F.Cu at (191.4, 44.2)

Commit message: ferrites and lna
Parts:
- added U11: LTC6400, Package_DFN_QFN:QFN-16-1EP_3x3mm_P0.5mm_EP1.7x1.7mm_ThermalVias, F.Cu at (180.7, 65.2)
- added U19: TO-252-5, Package_TO_SOT_SMD:TO-252-5_TabPin3, F.Cu at (77.5, 120.9)
- added U23: LTC6400, Package_DFN_QFN:QFN-16-1EP_3x3mm_P0.5mm_EP1.7x1.7mm_ThermalVias, F.Cu at (180.7, 83.2)
- added U27: TO-252-3, Package_TO_SOT_SMD:TO-252-3_TabPin2, F.Cu at (185.2, 146.2)
- added U31: TO-252-5, Package_TO_SOT_SMD:TO-252-5_TabPin3, F.Cu at (164.8, 146.5)
- L14, L16, L21, L44, L45, L6: moved to B.Cu
- moved L20 180.0 mm to (68.2, 124.4)
- moved L12 170.0 mm to (77.0, 108.2)
- moved L15 169.1 mm to (77.0, 110.6)
- moved L23 165.3 mm to (87.8, 111.0)
- moved L32 157.8 mm to (97.4, 123.6), turned to 90 degrees
- moved L24 150.0 mm to (108.4, 123.6), turned to 90 degrees
- moved L21 146.3 mm to (111.0, 112.4), turned to 180 degrees
- moved L30 120.5 mm to (160.4, 149.1), turned to 90 degrees
- moved L14 118.4 mm to (122.4, 39.6), turned to -90 degrees
- moved L22 115.8 mm to (172.6, 145.2)
- moved L2 113.3 mm to (121.0, 48.6)
- moved L1 113.2 mm to (121.0, 50.8)
- moved L42 89.0 mm to (169.8, 97.6)
- moved L33 86.4 mm to (190.0, 135.2), turned to 90 degrees
- moved L44 85.7 mm to (168.6, 92.4), turned to 180 degrees
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