File: angelia.kicad_sch (KiCad schematic)
At the start: 476 parts, among them J10 Conn_Coaxial, J15 Conn_02x05_Top_Bottom, J16 Conn_02x13_Top_Bottom, J18 Conn_02x05_Top_Bottom, J25 Conn_Coaxial, J3 Conn_Coaxial, J33 ATX-20, J5 Conn_Coaxial, J7 RJ45, P1 Conn_02x05_Top_Bottom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

Commit message: all resistors are not futile
Parts:
- added R128, R139: 5K11, Resistor_SMD:R_0805_2012Metric, symbol Device:R_Small
Changed lines of the file:
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@@
+    )
+  )
+  (symbol (lib_id "Device:R_Small") (at 24.13 61.595 0) (unit 1)
+    (in_bom yes) (on_board yes) (dnp no) (fields_autoplaced)
+    (property "Reference" "R139" (at 25.6286 60.9513 0)
+      (effects (font (size 1.27 1.27)) (justify left))
+    )
+    (property "Value" "5K11" (at 25.6286 62.8723 0)
+      (effects (font (size 1.27 1.27)) (justify left))
+    )
+    (property "Footprint" "Resistor_SMD:R_0805_2012Metric" (at 24.13 61.595 0)
+      (effects (font (size 1.27 1.27)) hide)
+    )
+    (property "Datasheet" "~" (at 24.13 61.595 0)
+      (effects (font (size 1.27 1.27)) hide)
+    )
+    (pin "1")
+    (pin "2")
+    (instances
+      (project "angelia"
+        (path "/2b733a3a-238e-4552-84a8-ec9891c3916f"
+          (reference "R139") (unit 1)
+        )
+      )
     )
   )
@@
         )
       )
+    )
+  )
+  (symbol (lib_id "Device:R_Small") (at 15.24 61.595 0) (unit 1)
+    (in_bom yes) (on_board yes) (dnp no) (fields_autoplaced)
+    (property "Reference" "R128" (at 16.7386 60.9513 0)
+      (effects (font (size 1.27 1.27)) (justify left))
+    )
+    (property "Value" "5K11" (at 16.7386 62.8723 0)
+      (effects (font (size 1.27 1.27)) (justify left))
+    )
+    (property "Footprint" "Resistor_SMD:R_0805_2012Metric" (at 15.24 61.595 0)
+      (effects (font (size 1.27 1.27)) hide)
+    )
+    (property "Datasheet" "~" (at 15.24 61.595 0)
+      (effects (font (size 1.27 1.27)) hide)
+    )
+    (pin "1")
+    (pin "2")
+    (instances
+      (project "angelia"
+        (path "/2b733a3a-238e-4552-84a8-ec9891c3916f"
+          (reference "R128") (unit 1)
+        )
+      )

Commit message: that's all folks
Parts:
- added R145: 4820P-1-104LF, Package_SO:SO-20_5.3x12.6mm_P1.27mm, symbol Device:R_Pack10
Changed lines of the file:
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@@
+    )
+  )
+  (symbol (lib_id "Device:R_Pack10") (at 59.055 60.96 0) (unit 1)
+    (in_bom yes) (on_board yes) (dnp no) (fields_autoplaced)
+    (property "Reference" "R145" (at 44.3231 60.3163 0)
+      (effects (font (size 1.27 1.27)) (justify right))
+    )
+    (property "Value" "4820P-1-104LF" (at 44.3231 62.2373 0)
+      (effects (font (size 1.27 1.27)) (justify right))
+    )
+    (property "Footprint" "Package_SO:SO-20_5.3x12.6mm_P1.27mm" (at 73.66 60.96 90)
+      (effects (font (size 1.27 1.27)) hide)
+    )
+    (property "Datasheet" "~" (at 59.055 60.96 0)
+      (effects (font (size 1.27 1.27)) hide)
+    )
+    (pin "1")
+    (pin "10")
+    (pin "11")
+    (pin "12")
+    (pin "13")
+    (pin "14")
+    (pin "15")
+    (pin "16")
+    (pin "17")
+    (pin "18")
+    (pin "19")
+    (pin "2")
+    (pin "20")
+    (pin "3")
+    (pin "4")
+    (pin "5")
+    (pin "6")
+    (pin "7")
+    (pin "8")
+    (pin "9")
+    (instances
+      (project "angelia"
+        (path "/2b733a3a-238e-4552-84a8-ec9891c3916f"
+          (reference "R145") (unit 1)
+        )
+      )
     )
   )
